Commit message: modified urdf

File: src/jimbo_navigation/urdf/jimbo_robot.urdf (robot description, URDF)
Before this commit: robot jimbo_robot, 6 links, 5 joints
Links:
- removed link caster_wheel
- link base_link: mass 5.0 -> 0.1; geometry collision box size=0.01 0.01 0.01; visual box size=0.01 0.01 0.01
- link camera_link: geometry visual box size=0.04 0.04 0.02
- link laser_frame: geometry visual cylinder length=0.02 radius=0.03
Joints:
- removed joint caster_wheel_joint
- joint camera_joint: origin xyz=0.1 0 0.08 rpy=0 0 0 -> xyz=0.05 0.255 -0.02 rpy=0 0 0
- joint left_wheel_joint: axis 0 0 1 -> 0 1 0; origin xyz=0 0.15 0 rpy=0 0 0 -> xyz=0 0.075 0 rpy=0 0 0
- joint lidar_joint: origin xyz=0 0 0.05 rpy=0 0 0 -> xyz=0 0.105 0.15 rpy=0 0 0
- joint right_wheel_joint: axis 0 0 1 -> 0 1 0; origin xyz=0 -0.15 0 rpy=0 0 0 -> xyz=0 -0.075 0 rpy=0 0 0

File: src/jimbo_navigation/urdf/jimbo_robot.urdf.xacro (robot description, xacro)
@@ -6,10 +6,10 @@
   <xacro:property name="base_height" value="0.01"/>
   <xacro:property name="wheel_radius" value="0.0635"/>
-  <xacro:property name="wheel_base" value="0.10"/> <!-- Small spacing between wheels -->
+  <xacro:property name="wheel_base" value="0.15"/> <!-- 15 cm spacing between wheels -->
   <!-- Sensor positions (relative to base_link, which is just a point) -->
-  <xacro:property name="lidar_x" value="-0.05"/> <!-- LiDAR to the left of wheels -->
-  <xacro:property name="lidar_z" value="0.08"/> <!-- LiDAR above wheels -->
-  <xacro:property name="camera_x" value="-0.07"/> <!-- Camera further left -->
-  <xacro:property name="camera_z" value="0.04"/> <!-- Camera below LiDAR -->
+  <xacro:property name="lidar_x" value="${wheel_base/2 + 0.03}"/> <!-- 3 cm left of left wheel -->
+  <xacro:property name="lidar_z" value="0.15"/> <!-- 15 cm above base -->
+  <xacro:property name="camera_x" value="${wheel_base/2 + 0.03 + 0.15}"/> <!-- 15 cm left of lidar -->
+  <xacro:property name="camera_z" value="-0.02"/> <!-- 2 cm below base -->
   <!-- Base link (just a point, no visible body) -->
   <link name="base_link">
@@ -35,5 +35,5 @@
   <link name="left_wheel">
     <visual>
-      <origin rpy="1.5708 1.5708 0"/>
+      <origin rpy="0 0 1.5708"/>
       <geometry>
         <cylinder radius="${wheel_radius}" length="0.04"/>
@@ -44,5 +44,5 @@
     </visual>
     <collision>
-      <origin rpy="0 1.5708 0"/>
+      <origin rpy="0 0 1.5708"/>
       <geometry>
         <cylinder radius="${wheel_radius}" length="0.04"/>
@@ -57,5 +57,5 @@
   <link name="right_wheel">
     <visual>
-      <origin rpy="1.5708 1.5708 0"/>
+      <origin rpy="0 0 1.5708"/>
       <geometry>
         <cylinder radius="${wheel_radius}" length="0.04"/>
@@ -66,5 +66,5 @@
     </visual>
     <collision>
-      <origin rpy="0 1.5708 0"/>
+      <origin rpy="0 0 1.5708"/>
       <geometry>
         <cylinder radius="${wheel_radius}" length="0.04"/>
@@ -76,22 +76,40 @@
     </inertial>
   </link>
-  <!-- LiDAR sensor (no geometry, just a frame) -->
-  <link name="laser_frame"/>
-  <!-- Camera sensor (no geometry, just a frame) -->
-  <link name="camera_link"/>
+  <!-- LiDAR sensor (now with a simple visual) -->
+  <link name="laser_frame">
+    <visual>
+      <geometry>
+        <cylinder radius="0.03" length="0.02"/>
+      </geometry>
+      <material name="green">
+        <color rgba="0.2 1 0.2 1"/>
+      </material>
+    </visual>
+  </link>
+  <!-- Camera sensor (now with a simple visual) -->
+  <link name="camera_link">
+    <visual>
+      <geometry>
+        <box size="0.04 0.04 0.02"/>
+      </geometry>
+      <material name="red">
+        <color rgba="1 0.2 0.2 1"/>
+      </material>
+    </visual>
+  </link>
   <!-- Joints -->
-  <!-- Left wheel joint: small spacing, left of base_link -->
+  <!-- Left wheel joint: left of base_link -->
   <joint name="left_wheel_joint" type="continuous">
     <parent link="base_link"/>
     <child link="left_wheel"/>
     <origin xyz="0 ${wheel_base/2} 0" rpy="0 0 0"/>
-    <axis xyz="0 0 1"/>
+    <axis xyz="0 1 0"/>
   </joint>
-  <!-- Right wheel joint: small spacing, right of base_link -->
+  <!-- Right wheel joint: right of base_link -->
   <joint name="right_wheel_joint" type="continuous">
     <parent link="base_link"/>
     <child link="right_wheel"/>
     <origin xyz="0 ${-wheel_base/2} 0" rpy="0 0 0"/>
-    <axis xyz="0 0 1"/>
+    <axis xyz="0 1 0"/>
   </joint>
   <!-- LiDAR joint: left and above wheels -->
@@ -101,5 +119,5 @@
     <origin xyz="${lidar_x} 0 ${lidar_z}" rpy="0 0 0"/>
   </joint>
-  <!-- Camera joint: below and left of LiDAR -->
+  <!-- Camera joint: left of lidar and below base -->
   <joint name="camera_joint" type="fixed">
     <parent link="base_link"/>

Commit message: updated robot launch file

File: src/jimbo_navigation/urdf/jimbo_robot.urdf (robot description, URDF)
Before this commit: robot jimbo_robot, 5 links, 4 joints
Links:
- removed link camera_link
- removed link laser_frame
- added link robot_camera_link; visual box size=0.04 0.04 0.02
- added link robot_lidar_link; visual cylinder length=0.02 radius=0.03
Joints:
- joint camera_joint: child camera_link -> robot_camera_link

Commit message: fixed transforms

File: src/jimbo_navigation/urdf/jimbo_robot.urdf (robot description, URDF)
Before this commit: robot jimbo_robot, 5 links, 4 joints
Links:
- removed link base_link
- added link robot_base_link, mass 0.1; collision box size=0.01 0.01 0.01; visual box size=0.01 0.01 0.01
Joints:
- joint camera_joint: parent base_link -> robot_base_link
- joint left_wheel_joint: parent base_link -> robot_base_link
- joint lidar_joint: child laser_frame -> robot_lidar_link; parent base_link -> robot_base_link
- joint right_wheel_joint: parent base_link -> robot_base_link
