Commit message: update

File: ros2_ws/src/jimbo_navigation/urdf/jimbo_robot_testbed.urdf (robot description, URDF)
Before this commit: robot jimbo_robot, 5 links, 4 joints
Links:
- link base_link: geometry collision box size=0.93 0.6 0.1; visual box size=0.93 0.6 0.1
- link left_wheel: geometry collision cylinder length=0.04 radius=0.0635; visual cylinder length=0.04 radius=0.0635
- link right_wheel: geometry collision cylinder length=0.04 radius=0.0635; visual cylinder length=0.04 radius=0.0635
Joints:
- joint left_wheel_joint: origin xyz=-(0.2325+0.16) (0.725/2) -0.1 rpy=0 0 0 -> xyz=0 0.32 -0.05 rpy=0 0 0
- joint lidar_joint: origin xyz=(0.2325+0.39) 0 0.06 rpy=0 0 0 -> xyz=0.435 0 0.06 rpy=0 0 0
- joint right_wheel_joint: origin xyz=-(0.2325+0.16) -(0.725/2) -0.1 rpy=0 0 0 -> xyz=0 -0.32 -0.05 rpy=0 0 0
